File: Circuit/bbesc_kiCad.kicad_pcb (KiCad board)
At the start: 2 copper layers, 110.5 x 82.5 mm, 82 parts, among them J1 CONN_01X02, J10 CONN_01X01, J11 CONN_01X01, J12 CONN_01X01, J13 CONN_01X01, J14 CONN_01X01, J15 CONN_01X02, J16 CONN_01X02, J17 CONN_01X01, J18 CONN_01X01, J19 CONN_01X01, J2 CONN_01X06, J3 CONN_01X06, J4 CONN_01X06, J5 CONN_01X02, J6 CONN_01X02, J7 CONN_01X01, J8 CONN_01X01, J9 RJ45, Q1 Q_NMOS_GDS, Q2 Q_NMOS_GDS, Q3 Q_NMOS_GDS, Q4 Q_NMOS_GDS, Q5 Q_NMOS_GDS, Q6 Q_NMOS_GDS, U1 teensy_3-2, U2 IR2101, U3 IR2101, U4 IR2101, U5 LM324N, U6 LM7805

Commit message: circuit for fab, foc bones
Parts:
- removed D4, D5: LED, LEDs:LED_1206
- removed J10, J11, J12, J13, J14, J17, J18, J19, J7, J8: CONN_01X01, Pin_Headers:Pin_Header_Straight_1x01_Pitch2.54mm
- removed J15, J16, J5, J6: CONN_01X02, Pin_Headers:Pin_Header_Straight_1x02_Pitch2.54mm
- removed J4: CONN_01X06, Pin_Headers:Pin_Header_Straight_1x06_Pitch2.54mm
- removed J9: RJ45, Connectors:RJ45_8
- removed R10: .001, R_SHUNT_3920:R_2816_HandSoldering
- removed R11, R12, R29: 470k, Resistors_SMD:R_1206_HandSoldering
- removed R19, R20: 4K7, Resistors_SMD:R_1206_HandSoldering
- removed R27: 12k, Resistors_SMD:R_1206_HandSoldering
- removed REF** (x3): MountingHole_3.2mm_M3, Mounting_Holes:MountingHole_3.2mm_M3
- added 3.3mm: MountingHole_3.2mm_M3, Mounting_Holes:MountingHole_3.2mm_M3, F.Cu at (164.2, 144.5)
- added ?: MountingHole_3.2mm_M3, Mounting_Holes:MountingHole_3.2mm_M3, F.Cu at (164.2, 73.4)
- added ?: MountingHole_3.2mm_M3, Mounting_Holes:MountingHole_3.2mm_M3, F.Cu at (81.0, 109.0)
- added C15: 10uF, Capacitors_SMD:C_1206_HandSoldering, B.Cu at (132.8, 132.0)
- added C16: 0.1uF, Capacitors_SMD:C_1206_HandSoldering, F.Cu at (130.3, 96.1)
- added C17: 2000uF, Capacitors_ThroughHole:CP_Radial_D13.0mm_P5.00mm, F.Cu at (112.4, 137.8)
- added C18: 10uF, Capacitors_SMD:C_1206_HandSoldering, F.Cu at (83.8, 85.6)
- added C19: 10uF, Capacitors_SMD:C_1206_HandSoldering, F.Cu at (89.7, 113.5)
- added C20: 10uF, Capacitors_SMD:C_1206_HandSoldering, F.Cu at (86.5, 78.9)
- added JP1: JUMPER, Pin_Headers:Pin_Header_Straight_1x02_Pitch2.54mm, F.Cu at (84.2, 100.7)
- added JP2: JUMPER3, Pin_Headers:Pin_Header_Straight_1x03_Pitch2.54mm, F.Cu at (81.2, 72.6)
- added P1: CONN_01X03, Pin_Headers:Pin_Header_Straight_1x03_Pitch2.54mm, F.Cu at (85.7, 73.0)
- added P2: CONN_01X06, Pin_Headers:Pin_Header_Straight_1x06_Pitch2.54mm, F.Cu at (94.6, 103.5)
- added P3: CONN_01X04, Pin_Headers:Pin_Header_Straight_1x04_Pitch2.54mm, F.Cu at (94.6, 107.3)
- added U7: INA21x, TO_SOT_Packages_SMD:SOT-363_SC-70-6_Handsoldering, F.Cu at (125.5, 124.0)
- added U8: TJA1051T-SN65HVD230D, Housings_SOIC:SOIC-8_3.9x4.9mm_Pitch1.27mm, F.Cu at (98.4, 113.7)
- C1, C2, C3: value 1uF -> 56uF; footprint Capacitors_SMD:C_1206_HandSoldering -> Capacitors_SMD:CP_Elec_6.3x7.7
- C10: moved to F.Cu
- C11: footprint Capacitors_THT:CP_Radial_D16.0mm_P7.50mm -> Capacitors_ThroughHole:CP_Radial_D13.0mm_P5.00mm
- C12: value 100pF -> 0.1uF; moved to F.Cu
- C13, C14: value 100pF -> 10uF
- Q2: footprint TO-251_IPAK_Vertical -> TO-251_IPAK_Slammed:TO-251_IPAK_Vertical
- R1, R2, R3, R4, R5, R6: value 470R -> 220R
- R13, R14, R15, R16, R17, R18: value 47R -> 4R7
- R7: value 12k -> 10K; moved to F.Cu
- R8: value 12k -> 47R; moved to F.Cu
- U5: value LM324N -> INA21x; footprint Housings_DIP:DIP-14_W7.62mm_Socket_LongPads -> TO_SOT_Packages_SMD:SOT-363_SC-70-6_Handsoldering
- moved R8 46.8 mm to (87.8, 76.2), turned to 0 degrees
- moved C12 37.9 mm to (130.3, 122.0)
- moved C14 31.1 mm to (132.7, 105.9), turned to 90 degrees
- moved J1 30.7 mm to (87.0, 143.5)
- moved C13 29.9 mm to (143.5, 79.9), turned to 90 degrees
- moved C10 28.2 mm to (89.5, 102.7)
- moved U6 25.7 mm to (87.1, 129.0)
- moved R6 25.4 mm to (123.8, 134.0)
- moved R7 25.2 mm to (93.2, 113.5)
- moved U1 21.4 mm to (96.5, 89.4)
- moved R4 19.5 mm to (123.8, 108.0)
- moved R3 18.9 mm to (123.8, 105.4)
- moved R5 17.3 mm to (123.8, 131.4)
- moved C11 12.8 mm to (98.4, 137.8)
- moved U5 9.30 mm to (125.3, 97.9), turned to 90 degrees
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Connections:
- net LO_B renamed LO_V
- net PHASE_C renamed PHASE_W
- net V_SENS_B renamed V_SENS_V
- C12 pad 1: A_SENS_B -> GND
- C12 pad 2: GND -> VCC
- C13 pad 1: A_SENS_A -> PHASE_U
- C13 pad 2: GND -> Net-(C13-Pad2)
- C14 pad 1: A_SENS_C -> PHASE_V
- C14 pad 2: GND -> Net-(C14-Pad2)
- C4 pad 1: PHASE_A -> PHASE_U
- C4 pad 2: Net-(C4-Pad2) -> Net-(C13-Pad2)
- C5 pad 1: PHASE_A -> PHASE_U
- C5 pad 2: Net-(C4-Pad2) -> Net-(C13-Pad2)
- C6 pad 1: PHASE_B -> PHASE_V
- C6 pad 2: Net-(C6-Pad2) -> Net-(C14-Pad2)
- C7 pad 1: PHASE_B -> PHASE_V
- C7 pad 2: Net-(C6-Pad2) -> Net-(C14-Pad2)
- D1 pad 1: Net-(C4-Pad2) -> Net-(C13-Pad2)
- D2 pad 1: Net-(C6-Pad2) -> Net-(C14-Pad2)
- J2 pad 4: Net-(J15-Pad1) -> MISO2
- J2 pad 5: Net-(J15-Pad2) -> MOSI2
- J3 pad 2: CS2 -> CS1
- J3 pad 4: Net-(J15-Pad1) -> MISO2
- J3 pad 5: Net-(J15-Pad2) -> MOSI2
- Q1 pad 3: PHASE_A -> PHASE_U
- Q2 pad 2: PHASE_A -> PHASE_U
- Q3 pad 3: PHASE_B -> PHASE_V
- Q4 pad 2: PHASE_B -> PHASE_V
- Q6 pad 3: Net-(Q6-Pad3) -> GND
- R1 pad 2: HI_A -> HI_U
- R2 pad 2: LO_A -> LO_U
- R21 pad 1: PHASE_A -> PHASE_U
- R21 pad 2: V_SENS_A -> V_SENS_U
- R22 pad 1: PHASE_B -> PHASE_V
- R23 pad 2: V_SENS_C -> V_SENS_W
- R24 pad 2: V_SENS_A -> V_SENS_U
- R26 pad 2: V_SENS_C -> V_SENS_W
- R3 pad 2: HI_B -> HI_V
- R5 pad 2: HI_C -> HI_W
- R6 pad 2: LO_C -> LO_W
- R7 pad 1: Net-(R11-Pad2) -> GND
- R7 pad 2: GND -> Net-(R7-Pad2)
- R8 pad 1: Net-(R12-Pad2) -> Net-(C20-Pad2)
- R8 pad 2: GND -> Net-(P1-Pad2)
- U1 pad 10: Net-(J5-Pad1) -> CS0
- U1 pad 15: CS2 -> CS1
- U1 pad 16: Net-(D4-Pad2) -> V_SENS_U
- U1 pad 17: V_SENS_A -> A_SENS_U
- U1 pad 19: V_SENS_C -> A_SENS_V
- U1 pad 20: CS1 -> LO_W
- U1 pad 21: A_SENS_A -> HI_V
- U1 pad 22: A_SENS_B -> HI_U
- U1 pad 23: A_SENS_C -> LO_U
- U1 pad 26: Net-(C10-Pad1) -> 5v
- U1 pad 3: LO_C -> CANTX
- U1 pad 4: HI_C -> CANRX
- U1 pad 6: HI_B -> HI_W
- U1 pad 9: Net-(J5-Pad2) -> CS2
- U2 pad 6: PHASE_A -> PHASE_U
- U2 pad 8: Net-(C4-Pad2) -> Net-(C13-Pad2)
- U3 pad 6: PHASE_B -> PHASE_V
- U3 pad 8: Net-(C6-Pad2) -> Net-(C14-Pad2)
- U5 pad 1: A_SENS_A -> GND
- U5 pad 2: Net-(R11-Pad2) -> GND
- U5 pad 3: Net-(Q2-Pad3) -> VCC
- U5 pad 4: VCC -> Net-(Q2-Pad3)
- U5 pad 5: Net-(Q4-Pad3) -> GND
- U5 pad 6: Net-(R27-Pad1) -> A_SENS_U
Routing:
- net PHASE_U: track 0.00 -> 116.5 mm
- net PHASE_A: track 113.0 -> 0.00 mm
- net V_SENS_C: track 104.5 -> 0.00 mm
- net PHASE_V: track 0.00 -> 99.6 mm
- net PHASE_B: track 95.7 -> 0.00 mm
- net V_SENS_W: track 0.00 -> 92.8 mm, vias 0 -> 3
- net Net-(Q6-Pad3): track 82.5 -> 0.00 mm
- net LO_W: track 0.00 -> 70.6 mm, vias 0 -> 2
- net VCC: track 94.4 -> 25.8 mm
- net A_SENS_A: track 61.1 -> 0.00 mm
- net V_SENS_A: track 58.2 -> 0.00 mm
- net A_SENS_V: track 0.00 -> 56.7 mm, vias 0 -> 1
- net A_SENS_C: track 52.5 -> 0.00 mm
- net HI_W: track 0.00 -> 50.4 mm, vias 0 -> 2
- net HI_B: track 44.6 -> 0.00 mm
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Other:
- board size 110.5 x 82.5 mm -> 90.8 x 78.7 mm
- net class Default: clearance 0.8 -> 0.15; trace_width 0.35 -> 0.4; via_dia 1 -> 1.2
- net class Drive: clearance 0.8 -> 0.2; via_dia 1 -> 1.2
- net class Phase: clearance 0.8 -> 0.2; via_dia 1 -> 1.2
- net class Phase Measurement: clearance 0.8 -> 0.2; via_dia 1 -> 1.2
- rule trace_clearance: 0.8 -> 0.15
- board text added: "+VE | -VE"
- board text added: "- s +"
- board text added: "3v3 | MOSI | MISO | SCK | CS1 | GND"
- board text added: "5 / 3 out"
- board text added: "FOCT v0.1"
- board text added: "GND | CANH | CANL | 3v3"
- board text added: "GND | CS_SLV | SCK | MOSI | MISO | 3v3"
- board text added: "github.com/jakeread/foct"

Commit message: circuit fab files v0.1
Parts:
- renumbered C11 to BFC11, C17 to BFC17, P3 to CANBUS, P1 to PWMIN, P2 to SPI1CS0, J3 to SPI2CS1, J2 to SPI2CS2, JP1 to TPWR
Routing:
- net Net-(Q4-Pad3): track 27.6 -> 84.0 mm
- net Net-(Q2-Pad3): track 26.7 -> 83.1 mm
Other:
- board text added: "+VE | GND"
- board text removed: "+VE | -VE"

Commit message: board v0.2
Parts:
- removed 3.3mm, ? (x2): MountingHole_3.2mm_M3, Mounting_Holes:MountingHole_3.2mm_M3
- removed BFC11, BFC17: 2000uF, Capacitors_ThroughHole:CP_Radial_D13.0mm_P5.00mm
- removed C1: 56uF, Capacitors_SMD:CP_Elec_6.3x7.7
- removed C8: 10uF, Capacitors_SMD:C_1206_HandSoldering
- removed CANBUS: CONN_01X04, Pin_Headers:Pin_Header_Straight_1x04_Pitch2.54mm
- removed D3: 1N4001, Diodes_SMD:D_SMA_Handsoldering
- removed JP2: JUMPER3, Pin_Headers:Pin_Header_Straight_1x03_Pitch2.54mm
- removed PWMIN: CONN_01X03, Pin_Headers:Pin_Header_Straight_1x03_Pitch2.54mm
- removed R1: 220R, Resistors_SMD:R_1206_HandSoldering
- removed SPI1CS0, SPI2CS1, SPI2CS2: CONN_01X06, Pin_Headers:Pin_Header_Straight_1x06_Pitch2.54mm
- removed TPWR: JUMPER, Pin_Headers:Pin_Header_Straight_1x02_Pitch2.54mm
- removed U1: teensy_3-2, teensy_3-2_bottomLess:Teensy3.2-bottomLess
- removed U4: IR2101, Housings_DIP:DIP-8_W7.62mm_Socket_LongPads
- removed U5, U7: INA21x, TO_SOT_Packages_SMD:SOT-363_SC-70-6_Handsoldering
- removed U6: LM7805, TO_SOT_Packages_THT:TO-220_Horizontal
- removed U8: TJA1051T-SN65HVD230D, Housings_SOIC:SOIC-8_3.9x4.9mm_Pitch1.27mm
- added C11: 22nF, Capacitors_SMD:C_1206_HandSoldering, F.Cu at (133.2, 97.8)
- added C17: 100nF, Capacitors_SMD:C_1206_HandSoldering, F.Cu at (145.7, 85.3)
- added C21: 2.2nF, Capacitors_SMD:C_1206_HandSoldering, F.Cu at (138.2, 114.3)
- added C22: 2.2nF, Capacitors_SMD:C_1206_HandSoldering, F.Cu at (138.2, 107.7)
- added C23: 2000uF, Capacitors_ThroughHole:CP_Radial_D13.0mm_P5.00mm, F.Cu at (115.1, 116.1)
- added C24: 100uF, Capacitors_SMD:CP_Elec_6.3x7.7, F.Cu at (145.7, 80.6)
- added C25: 2000uF, Capacitors_ThroughHole:CP_Radial_D13.0mm_P5.00mm, F.Cu at (128.4, 116.1)
- added C26: 10uF, Capacitors_SMD:C_1206_HandSoldering, B.Cu at (145.2, 97.3)
- added C29: 10uF, Capacitors_SMD:C_1206_HandSoldering, B.Cu at (145.2, 88.8)
- added C30: 10uF, Capacitors_SMD:C_1206_HandSoldering, B.Cu at (143.3, 88.8)
- added C31: 10uF, Capacitors_SMD:C_1206_HandSoldering, B.Cu at (141.4, 88.8)
- added J3: CONN_01X02, Wire_Connections_Bridges:WireConnection_2.50mmDrill_LargePad, F.Cu at (104.1, 125.6)
- added JP1: JUMPER, Pin_Headers:Pin_Header_Straight_1x02_Pitch2.54mm, F.Cu at (123.3, 78.1)
- added JP3: JUMPER3, Pin_Headers:Pin_Header_Straight_1x03_Pitch2.54mm, F.Cu at (99.8, 75.6)
- added L1: 22uH, Inductors:Inductor_Taiyo-Yuden_NR-40xx_HandSoldering, F.Cu at (145.0, 74.8)
- added P2: CONN_01X03, Pin_Headers:Pin_Header_Straight_1x03_Pitch2.54mm, F.Cu at (99.8, 88.4)
- added R10: 1M, Resistors_SMD:R_1206_HandSoldering, F.Cu at (139.1, 85.3)
- added R11: 100R, Resistors_SMD:R_1206_HandSoldering, F.Cu at (142.5, 115.3)
- added R12: 100R, Resistors_SMD:R_1206_HandSoldering, F.Cu at (142.5, 113.1)
- added R19: 39K, Resistors_SMD:R_1206_HandSoldering, B.Cu at (151.6, 79.8)
- added R20: 5K6, Resistors_SMD:R_1206_HandSoldering, B.Cu at (151.6, 77.7)
- added R27: 4R7, Resistors_SMD:R_1206_HandSoldering, B.Cu at (159.8, 108.8)
- added R29: 39k, Resistors_SMD:R_1206_HandSoldering, B.Cu at (162.9, 123.0)
- added R30: 39K, Resistors_SMD:R_1206_HandSoldering, B.Cu at (151.4, 113.3)
- added R31: 5K6, Resistors_SMD:R_1206_HandSoldering, B.Cu at (151.4, 111.1)
- added REF**: MountingHole_3.2mm_M3_ISO14580, Mounting_Holes:MountingHole_3.2mm_M3_ISO14580, F.Cu at (168.0, 70.2)
- added REF**: MountingHole_3.2mm_M3_ISO14580, Mounting_Holes:MountingHole_3.2mm_M3_ISO14580, F.Cu at (100.1, 70.2)
- added REF**: MountingHole_3.2mm_M3_ISO14580, Mounting_Holes:MountingHole_3.2mm_M3_ISO14580, F.Cu at (135.0, 127.4)
- C10: value 10uF -> 2.2uF
- C12: value 0.1uF -> 10uF; moved to B.Cu
- C16: value 0.1uF -> 10uF
- C18, C19, C20: value 10uF -> 220nF
- C2: value 56uF -> 10uF; footprint Capacitors_SMD:CP_Elec_6.3x7.7 -> Capacitors_SMD:C_1206_HandSoldering
- C3: value 56uF -> 10uF; footprint Capacitors_SMD:CP_Elec_6.3x7.7 -> Capacitors_SMD:C_1206_HandSoldering; moved to B.Cu
- C4: value 10uF -> 2.2uF; moved to F.Cu
- C5, C7: value 0.1uF -> 2.2uF; moved to F.Cu
- C6: value 10uF -> 120pF; moved to F.Cu
- C9: value 0.1uF -> 6.8nF; moved to F.Cu
- D1: value 1N4001 -> DIODESCH
- D2: value 1N4001 -> TVS 5v
- J1: value CONN_01X02 -> CONN_01X06; footprint Wire_Connections_Bridges:WireConnection_2.50mmDrill_LargePad -> Pin_Headers:Pin_Header_Straight_1x06_Pitch2.54mm
- Q1, Q2, Q3, Q4, Q5, Q6: footprint TO-251_IPAK_Slammed:TO-251_IPAK_Vertical -> HTO-252:TO-252-2; moved to B.Cu
- R13, R14: value 4R7 -> 100R
- R15, R26: moved to B.Cu
- R17: value 4R7 -> 39k; moved to B.Cu
- R18: value 4R7 -> SHNT; footprint Resistors_SMD:R_1206_HandSoldering -> R_SHUNT_3920:R_SHUNT_3920; moved to B.Cu
- R2: value 220R -> 47R
- R21: value 39K -> 4R7; moved to B.Cu
- R22: value 39K -> 4R7
- R23: value 39K -> 39k; moved to B.Cu
- R24: value 5K6 -> SHNT; footprint Resistors_SMD:R_1206_HandSoldering -> R_SHUNT_3920:R_SHUNT_3920; moved to B.Cu
- R25: value 5K6 -> 39K; moved to B.Cu
- R28: value .001 -> 4R7; footprint R_SHUNT_3920:R_2816_HandSoldering -> Resistors_SMD:R_1206_HandSoldering; moved to F.Cu
- R3: value 220R -> 18k; moved to F.Cu
- R4, R6: value 220R -> 3k3; moved to F.Cu
- R5: value 220R -> 10k; moved to F.Cu
- R7: value 10K -> 3k3
- R8: value 47R -> 15k
- R9: value .001 -> 220k; footprint R_SHUNT_3920:R_2816_HandSoldering -> Resistors_SMD:R_1206_HandSoldering; moved to F.Cu
- U2: value IR2101 -> teensy_3-2; footprint Housings_DIP:DIP-8_W7.62mm_Socket_LongPads -> teensy_3-2_bottomLess:Teensy3.2-bottomLess
- U3: value IR2101 -> DRV_8302; footprint Housings_DIP:DIP-8_W7.62mm_Socket_LongPads -> HTSSOP-56:TSSOP-56_6.1x14mm_Pitch0.5mm
- moved C20 79.7 mm to (156.3, 117.4), turned to 180 degrees
- moved C18 72.4 mm to (156.2, 83.4), turned to 180 degrees
- moved C19 67.7 mm to (156.1, 100.5), turned to 180 degrees
- moved C3 52.0 mm to (109.7, 81.9)
- moved C9 49.5 mm to (130.6, 82.9)
- moved R26 49.1 mm to (151.3, 94.9), turned to 0 degrees
- moved R8 44.2 mm to (130.5, 87.4)
- moved R7 42.5 mm to (130.6, 93.2)
- moved R5 42.3 mm to (123.6, 89.2), turned to 90 degrees
- moved C10 42.0 mm to (131.4, 105.7), turned to 180 degrees
- moved R23 41.6 mm to (162.8, 106.1)
- moved R17 41.5 mm to (162.8, 89.1)
- moved R6 41.1 mm to (128.2, 93.2), turned to 90 degrees
- moved J1 39.7 mm to (99.8, 105.9), turned to 180 degrees
- moved R13 35.7 mm to (142.5, 108.7)
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Connections:
- C12 pad 1: GND -> VCC
- C12 pad 2: VCC -> GND
- C13 pad 1: PHASE_U -> VCC
- C13 pad 2: Net-(C13-Pad2) -> GND
- C14 pad 1: PHASE_V -> VCC
- C14 pad 2: Net-(C14-Pad2) -> GND
- C15 pad 1: PHASE_W -> VCC
- C15 pad 2: Net-(C15-Pad2) -> GND
- C18 pad 1: GND -> PHASE_U
- C18 pad 2: 3v3 -> Net-(C18-Pad2)
- C19 pad 1: VCC -> PHASE_V
- C19 pad 2: GND -> Net-(C19-Pad2)
- C2 pad 1: VCC -> GND
- C2 pad 2: GND -> 3v3
- C20 pad 1: GND -> PHASE_W
- C3 pad 1: VCC -> GND
- C3 pad 2: GND -> SIMPLE_INPUT
- C4 pad 1: PHASE_U -> Net-(C4-Pad1)
- C4 pad 2: Net-(C13-Pad2) -> GND
- C5 pad 1: PHASE_U -> Net-(C4-Pad1)
- C5 pad 2: Net-(C13-Pad2) -> GND
- C6 pad 1: PHASE_V -> Net-(C6-Pad1)
- C6 pad 2: Net-(C14-Pad2) -> GND
- C7 pad 1: PHASE_V -> Net-(C7-Pad1)
- C7 pad 2: Net-(C14-Pad2) -> GND
- C9 pad 1: PHASE_W -> Net-(C9-Pad1)
- C9 pad 2: Net-(C15-Pad2) -> GND
- D1 pad 1: Net-(C13-Pad2) -> Net-(C17-Pad1)
- D1 pad 2: VCC -> GND
- D2 pad 1: Net-(C14-Pad2) -> 5v
- D2 pad 2: VCC -> GND
- J1 pad 2: VCC -> CS2
- Q2 pad 3: Net-(Q2-Pad3) -> GND
- Q4 pad 3: Net-(Q4-Pad3) -> /H_V_LO
- Q6 pad 3: GND -> /H_W_LO
- R13 pad 1: Net-(Q1-Pad1) -> /SHNT_V_HI
- R13 pad 2: Net-(R13-Pad2) -> Net-(C22-Pad2)
- R14 pad 1: Net-(Q2-Pad1) -> /SHNT_V_LO
- R14 pad 2: Net-(R14-Pad2) -> Net-(C22-Pad1)
- R15 pad 1: Net-(Q3-Pad1) -> Net-(Q1-Pad1)
- R15 pad 2: Net-(R15-Pad2) -> DRV_HI_U
- R16 pad 1: Net-(Q4-Pad1) -> Net-(Q2-Pad1)
- R16 pad 2: Net-(R16-Pad2) -> DRV_LO_U
- R17 pad 1: Net-(Q5-Pad1) -> GND
- R17 pad 2: Net-(R17-Pad2) -> Net-(Q2-Pad1)
- R18 pad 1: Net-(Q6-Pad1) -> /H_V_LO
- R18 pad 2: Net-(R18-Pad2) -> GND
- R2 pad 1: Net-(R2-Pad1) -> SIMPLE_INPUT
- R2 pad 2: LO_U -> Net-(P2-Pad2)
- R21 pad 1: PHASE_U -> Net-(Q3-Pad1)
- R21 pad 2: V_SENS_U -> DRV_HI_V
- R22 pad 1: PHASE_V -> Net-(Q4-Pad1)
- R22 pad 2: V_SENS_V -> DRV_LO_V
- R23 pad 1: PHASE_W -> /H_V_LO
- R23 pad 2: V_SENS_W -> Net-(Q4-Pad1)
- R24 pad 1: GND -> /H_W_LO
- R24 pad 2: V_SENS_U -> GND
- R25 pad 1: GND -> PHASE_V
- R26 pad 1: GND -> V_SENS_V
- R26 pad 2: V_SENS_W -> GND
- R28 pad 1: Net-(Q4-Pad3) -> Net-(Q6-Pad1)
- R28 pad 2: GND -> DRV_LO_W
- R3 pad 2: HI_V -> 5v
- R4 pad 1: Net-(R4-Pad1) -> GND
- R4 pad 2: LO_V -> Net-(R3-Pad1)
- R5 pad 2: HI_W -> 5v
- R6 pad 1: Net-(R6-Pad1) -> GND
- R6 pad 2: LO_W -> Net-(R6-Pad2)
- R8 pad 1: Net-(C20-Pad2) -> Net-(C6-Pad1)
- R8 pad 2: Net-(P1-Pad2) -> Net-(C9-Pad1)
- R9 pad 1: Net-(Q2-Pad3) -> Net-(R9-Pad1)
- U2 pad 1: VCC -> Net-(U2-Pad1)
- U2 pad 2: Net-(R1-Pad1) -> EN_GATE
- U2 pad 3: Net-(R2-Pad1) -> CANTX
- U2 pad 4: GND -> CANRX
- U2 pad 5: Net-(R14-Pad2) -> MC_LO_V
- U2 pad 6: PHASE_U -> MC_HI_W
- U2 pad 7: Net-(R13-Pad2) -> MOSI2
- U2 pad 8: Net-(C13-Pad2) -> MISO2
- U3 pad 1: VCC -> Net-(R9-Pad1)
- U3 pad 2: Net-(R3-Pad1) -> Net-(C6-Pad1)
- U3 pad 3: Net-(R4-Pad1) -> Net-(R3-Pad1)
- U3 pad 4: GND -> Net-(U3-Pad4)
- U3 pad 5: Net-(R16-Pad2) -> Net-(U3-Pad5)
- U3 pad 6: PHASE_V -> DRV_FAULT
- U3 pad 7: Net-(R15-Pad2) -> Net-(R6-Pad2)
- U3 pad 8: Net-(C14-Pad2) -> Net-(R7-Pad2)
Routing:
- net PHASE_U: track 116.5 -> 27.4 mm
- net Net-(Q4-Pad3): track 84.0 -> 0.00 mm, vias 1 -> 0
- net Net-(Q2-Pad3): track 83.1 -> 0.00 mm, vias 1 -> 0
- net PHASE_V: track 99.6 -> 28.5 mm
- net LO_W: track 70.6 -> 0.00 mm, vias 2 -> 0
- net DRV_FAULT: track 0.00 -> 60.6 mm, vias 0 -> 3
- net PHASE_W: track 99.6 -> 43.4 mm
- net GND: track 102.1 -> 50.4 mm, vias 2 -> 6
- net HI_W: track 50.4 -> 0.00 mm, vias 2 -> 0
- net /H_W_LO: track 0.00 -> 44.7 mm, vias 0 -> 1
- net EN_GATE: track 0.00 -> 42.6 mm, vias 0 -> 1
- net MC_LO_V: track 0.00 -> 42.5 mm, vias 0 -> 1
- net MC_AREF: track 0.00 -> 42.2 mm, vias 0 -> 2
- net MC_HI_W: track 0.00 -> 41.7 mm, vias 0 -> 2
- net DRV_LO_W: track 0.00 -> 40.8 mm
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- added copper zone on B.Cu, net /H_V_LO
- added copper zone on B.Cu, net /H_W_LO
- added copper zone on B.Cu, net PHASE_U
- added copper zone on B.Cu, net PHASE_V
- added copper zone on B.Cu, net PHASE_W
Other:
- board size 90.8 x 78.7 mm -> 74.3 x 63.5 mm
- net class Default: clearance 0.15 -> 0.2; trace_width 0.4 -> 0.25; via_dia 1.2 -> 0.7; via_drill 0.8 -> 0.4
- net class Drive: trace_width 0.8 -> 0.25; via_dia 1.2 -> 0.7; via_drill 0.8 -> 0.4
- net class Phase: trace_width 1.5 -> 0.25; via_dia 1.2 -> 0.7; via_drill 0.8 -> 0.4
- net class Phase Measurement: trace_width 0.35 -> 0.4; via_dia 1.2 -> 0.7; via_drill 0.8 -> 0.4
- rule trace_clearance: 0.15 -> 0.2
- board text added: "FOCT v0.2"
- board text added: "U"
- board text added: "V"
- board text added: "W"
- board text added: "field oriented control on teensy"
- board text removed: "FOCT v0.1"
- board text removed: "GND | CANH | CANL | 3v3"
- board text removed: "GND | CS_SLV | SCK | MOSI | MISO | 3v3"

Commit message: documentation
Parts:
- removed R23, R29: 39k, Resistors_SMD:R_1206_HandSoldering
- removed REF** (x3): MountingHole_3.2mm_M3_ISO14580, Mounting_Holes:MountingHole_3.2mm_M3_ISO14580
- added C27: 10uF, Capacitors_SMD:C_1206_HandSoldering, B.Cu at (167.3, 95.3)
- added C28: 10uF, Capacitors_SMD:C_1206_HandSoldering, B.Cu at (167.3, 110.6)
- added C32: 100uF, Capacitors_SMD:CP_Elec_6.3x7.7, F.Cu at (148.0, 106.5)
- added C8: 2.2uF, Capacitors_SMD:C_1206_HandSoldering, B.Cu at (137.2, 91.3)
- added M3: MountingHole_3.2mm_M3_DIN965_Pad, Mounting_Holes:MountingHole_3.2mm_M3_DIN965_Pad, F.Cu at (100.3, 127.0)
- added M3 -> 81.28mm: MountingHole_3.2mm_M3_DIN965_Pad, Mounting_Holes:MountingHole_3.2mm_M3_DIN965_Pad, F.Cu at (156.8, 127.0)
- added M3 56.515mm Square: MountingHole_3.2mm_M3_DIN965_Pad, Mounting_Holes:MountingHole_3.2mm_M3_DIN965_Pad, F.Cu at (156.8, 70.5)
- added M3 offset inside by 3.429mm: MountingHole_3.2mm_M3_DIN965_Pad, Mounting_Holes:MountingHole_3.2mm_M3_DIN965_Pad, F.Cu at (100.3, 70.5)
- added P5: CONN_01X01, Mounting_Holes:MountingHole_2.7mm_Pad_Via, F.Cu at (172.7, 87.2)
- added P6: CONN_01X01, Mounting_Holes:MountingHole_2.7mm_Pad_Via, F.Cu at (172.7, 102.4)
- added P7: CONN_01X01, Mounting_Holes:MountingHole_2.7mm_Pad_Via, F.Cu at (172.7, 117.7)
- C10, C11, C4, C5, C7, R16, R22: moved to B.Cu
- C12: value 10uF -> 1uF
- C15: value 10uF -> 15uF
- R17: value 39k -> 10k; moved to F.Cu
- moved R17 36.3 mm to (130.2, 73.2), turned to 0 degrees
- moved C26 28.2 mm to (167.2, 79.6), turned to 0 degrees
- moved R25 19.5 mm to (146.6, 78.1)
- moved R26 19.5 mm to (146.6, 75.9)
- moved C20 18.1 mm to (151.8, 99.8)
- moved R31 14.3 mm to (142.3, 122.1)
- moved R30 14.2 mm to (142.3, 124.2)
- moved R22 13.0 mm to (150.2, 109.0), turned to 90 degrees
- moved C7 12.8 mm to (135.1, 91.3), turned to 90 degrees
- moved C4 12.6 mm to (134.8, 96.0), turned to 180 degrees
- moved R28 12.1 mm to (152.0, 117.7), turned to 90 degrees
- moved R16 11.0 mm to (151.9, 90.7), turned to 270 degrees
- moved C5 10.0 mm to (134.8, 98.0), turned to 180 degrees
- moved R20 8.77 mm to (146.5, 70.6)
- moved R19 8.69 mm to (146.5, 72.7)
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Connections:
- P2 pad 2: Net-(P2-Pad2) -> Net-(JP3-Pad2)
- P2 pad 3: Net-(JP3-Pad2) -> Net-(P2-Pad3)
- R17 pad 1: GND -> 5v
- R17 pad 2: Net-(Q2-Pad1) -> DRV_FAULT
- R2 pad 2: Net-(P2-Pad2) -> Net-(P2-Pad3)
- U3 pad 44: /H_U_LO -> GND
Routing:
- net DC_CAL: track 31.5 -> 91.0 mm, vias 1 -> 3
- net DRV_FAULT: track 60.6 -> 88.6 mm, vias 3 -> 2
- net V_SENS_U: track 39.3 -> 59.5 mm, vias 1 -> 3
- net PHASE_V: track 28.5 -> 48.6 mm, vias 0 -> 3
- net Net-(C7-Pad1): track 23.8 -> 4.68 mm, vias 2 -> 1
- net /H_W_LO: track 44.7 -> 26.0 mm
- net /H_V_LO: track 30.4 -> 12.4 mm
- net DRV_LO_W: track 40.8 -> 23.0 mm
- net Net-(C20-Pad2): track 25.6 -> 8.55 mm, vias 0 -> 2
- net /H_U_LO: track 15.2 -> 0.00 mm, vias 3 -> 0
- net DRV_LO_U: track 19.4 -> 5.28 mm, vias 0 -> 1
- net Net-(C4-Pad1): track 32.3 -> 18.5 mm, vias 0 -> 2
- net VCC: track 23.4 -> 34.9 mm
- net V_SENS_W: track 52.7 -> 41.4 mm, vias 2 -> 1
- net DRV_LO_V: track 26.5 -> 15.4 mm, vias 0 -> 1
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Other:
- board size 74.3 x 63.5 mm -> 81.4 x 63.5 mm
- net class Default: clearance 0.2 -> 0.175; via_dia 0.7 -> 0.8
- net class Drive: clearance 0.2 -> 0.175; trace_width 0.25 -> 0.6; via_dia 0.7 -> 1.2; via_drill 0.4 -> 0.8
- net class Phase: clearance 0.2 -> 0.175; via_dia 0.7 -> 0.8
- net class Phase Measurement: clearance 0.2 -> 0.175; via_dia 0.7 -> 0.8
- rule trace_clearance: 0.2 -> 0.175
- board text added: "- + s"
- board text added: "<- IRLR2905Z"
- board text added: "DRV8302 ->"
- board text added: "FOCT v0.3"
- board text removed: "- s +"
- board text removed: "FOCT v0.2"
